File: Hardware/SparkFun_DataLogger_IoT_9DOF.brd (EAGLE design)
At the start: 50.8 x 38.1 mm, 158 parts, among them J10 QWIIC_RIGHT_ANGLE, J3 MICRO-SD-PUSH-PUSH-EXT-PIN, J4 Vertical Qwiic Connector, U1 ESP-WROOM-32E, U10 74HC4066_QUAD_BILATERAL_SWITC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, U2 CH340C, U3 XC6222B331MR-G, U4 MAX17048, U5 MCP73831, U6 XC6222B331MR-G, U7 ISM330DHCX, U8 MMC5983MA_QFN16, U9 74HC4066_QUAD_BILATERAL_SWITC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

Commit message: v11 - SparkFun_DataLogger_IoT_9DOF
Parts:
- removed U$39: (no value), output:ESP320
- added U$50: (no value), output:DATALOGGER0
- added U$51: (no value), output:DATALOGGER1
- U$1: device output:OPENLOG0 -> output:IOT_9DOF0
- U$44: device output:OPENLOG_ESP320 -> output:IOT_9DOF10
- moved U$1 2.22 mm to (39.2, 24.1)
- moved U$44 0.76 mm to (25.4, 20.8)
- moved U$14 0.40 mm to (46.0, 26.8)
- moved U$13 0.38 mm to (47.5, 25.3)
- moved U$15 0.38 mm to (46.0, 25.3)
Other:
- board text added: "v11"
- board text removed: "v10"
Changed lines of the file:
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@@
 <drawing>
 <settings>
-<setting alwaysvectorfont="yes"/>
+<setting alwaysvectorfont="no"/>
 <setting verticaltext="up"/>
 </settings>
@@
 <wire x1="6.0325" y1="33.3375" x2="6.6675" y2="33.9725" width="0.2032" layer="21"/>
 <wire x1="6.0325" y1="33.9725" x2="6.6675" y2="33.3375" width="0.2032" layer="21"/>
-<wire x1="44.45" y1="25.019" x2="44.45" y2="27.051" width="0.2032" layer="21"/>
-<wire x1="44.45" y1="27.051" x2="44.069" y2="26.162" width="0.2032" layer="21"/>
-<circle x="44.45" y="24.13" radius="0.508" width="0.2032" layer="21"/>
-<wire x1="44.45" y1="27.051" x2="44.831" y2="26.162" width="0.2032" layer="21"/>
-<wire x1="45.339" y1="24.13" x2="47.371" y2="24.13" width="0.2032" layer="21"/>
-<wire x1="47.371" y1="24.13" x2="46.482" y2="24.511" width="0.2032" layer="21"/>
-<wire x1="47.371" y1="24.13" x2="46.482" y2="23.749" width="0.2032" layer="21"/>
-<circle x="44.45" y="24.13" radius="0.1016" width="0.2032" layer="21"/>
+<wire x1="44.831" y1="25.019" x2="44.831" y2="27.051" width="0.2032" layer="21"/>
+<wire x1="44.831" y1="27.051" x2="44.45" y2="26.162" width="0.2032" layer="21"/>
+<circle x="44.831" y="24.13" radius="0.508" width="0.2032" layer="21"/>
+<wire x1="44.831" y1="27.051" x2="45.212" y2="26.162" width="0.2032" layer="21"/>
+<wire x1="45.72" y1="24.13" x2="47.752" y2="24.13" width="0.2032" layer="21"/>
+<wire x1="47.752" y1="24.13" x2="46.863" y2="24.511" width="0.2032" layer="21"/>
+<wire x1="47.752" y1="24.13" x2="46.863" y2="23.749" width="0.2032" layer="21"/>
+<circle x="44.831" y="24.13" radius="0.1016" width="0.2032" layer="21"/>
 <wire x1="2.54" y1="11.43" x2="2.54" y2="12.7" width="0.2032" layer="21"/>
 <wire x1="1.905" y1="12.065" x2="3.175" y2="12.065" width="0.2032" layer="21"/>
@@
 White Silkscreen
 </text>
-<text x="45.72" y="0.381" size="1.778" layer="16" font="vector" ratio="15" rot="SMR0" align="bottom-center">v10</text>
+<text x="45.72" y="0.381" size="1.778" layer="16" font="vector" ratio="15" rot="SMR0" align="bottom-center">v11</text>
 <text x="-1.27" y="43.18" size="1.778" layer="47" font="vector" ratio="15" align="bottom-right">Dimensions
 In Inches</text>
@@
 <element name="U$11" library="output" package="Y0" value="" x="7.493" y="36.195" smashed="yes"/>
 <element name="U$12" library="output" package="Z0" value="" x="7.493" y="34.798" smashed="yes"/>
-<element name="U$13" library="output" package="X0" value="" x="47.117" y="25.273" smashed="yes"/>
-<element name="U$14" library="output" package="Y0" value="" x="45.593" y="26.67" smashed="yes"/>
-<element name="U$15" library="output" package="Z0" value="" x="45.593" y="25.273" smashed="yes"/>
+<element name="U$13" library="output" package="X0" value="" x="47.498" y="25.273" smashed="yes"/>
+<element name="U$14" library="output" package="Y0" value="" x="45.974" y="26.797" smashed="yes"/>
+<element name="U$15" library="output" package="Z0" value="" x="45.974" y="25.273" smashed="yes"/>
 <element name="U$16" library="output" package="##RESET##0" value="" x="48.768" y="36.83" smashed="yes" rot="MR0"/>
 <element name="U$17" library="output" package="#0_#_#BOOT##0" value="" x="48.768" y="34.29" smashed="yes" rot="MR0"/>
@@
 <element name="U$43" library="output" package="#35#0" value="" x="18.288" y="25.4" smashed="yes" rot="MR0"/>
 <element name="LOGO4" library="SparkFun-Aesthetics" package="OSHW-LOGO-S" value="OSHW-LOGOS" x="25.4" y="17.78" smashed="yes" rot="MR0"/>
-<element name="U$44" library="output" package="OPENLOG_ESP320" value="" x="25.4" y="21.59" smashed="yes" rot="MR0"/>
 <element name="U$45" library="output" package="#SHLD#0" value="" x="34.798" y="5.842" smashed="yes" rot="MR0"/>
 <element name="U$46" library="output" package="#I�C#0" value="" x="36.83" y="11.4935" smashed="yes" rot="MR0"/>
@@
 <element name="LOGO6" library="SparkFun-Aesthetics" package="SFE_LOGO_FLAME_.2" value="SFE_LOGO_FLAME.2_INCH" x="45.466" y="17.78" smashed="yes"/>
 <element name="IMU_INT1" library="SparkFun-Connectors" package="PAD.03X.05" value="TEST-POINT3X5" x="11.43" y="35.56" smashed="yes" rot="MR0"/>
-<element name="U$1" library="output" package="OPENLOG0" value="" x="38.1" y="26.035" smashed="yes"/>
-<element name="U$39" library="output" package="ESP320" value="" x="38.1" y="24.4475" smashed="yes"/>
+<element name="U$50" library="output" package="DATALOGGER0" value="" x="39.243" y="25.654" smashed="yes"/>
+<element name="U$51" library="output" package="DATALOGGER1" value="" x="25.4" y="22.86" smashed="yes" rot="MR0"/>
+<element name="U$1" library="output" package="IOT_9DOF0" value="" x="39.243" y="24.13" smashed="yes"/>
+<element name="U$44" library="output" package="IOT_9DOF10" value="" x="25.4" y="20.828" smashed="yes" rot="MR0"/>
 </elements>
 <signals>
@@
 <wire x1="17.5006" y1="31.4706" x2="26.9494" y2="31.4706" width="0.1524" layer="16"/>
 <via x="19.685" y="17.526" extent="1-16" drill="0.3"/>
-<via x="35.8418" y="25.4" extent="1-16" drill="0.3"/>
+<via x="35.8418" y="24.892" extent="1-16" drill="0.3"/>
 <via x="48.2878" y="25.4" extent="1-16" drill="0.3"/>
-<wire x1="35.8418" y1="25.4" x2="48.2878" y2="25.4" width="0.1524" layer="16"/>
+<wire x1="48.2878" y1="25.4" x2="36.3498" y2="25.4" width="0.1524" layer="16"/>
+<wire x1="36.3498" y1="25.4" x2="35.8418" y2="24.892" width="0.1524" layer="16"/>
 <via x="42.672" y="15.367" extent="1-16" drill="0.3"/>
 <wire x1="40.39" y1="12.62" x2="40.39" y2="11.434" width="0.254" layer="1"/>
@@
 <via x="20.447" y="23.622" extent="1-16" drill="0.3"/>
 <wire x1="20.447" y1="23.622" x2="20.447" y2="21.717" width="0.4064" layer="1"/>
-<via x="27.94" y="23.368" extent="1-16" drill="0.3"/>
-<via x="27.94" y="24.892" extent="1-16" drill="0.3"/>
-<wire x1="27.94" y1="24.892" x2="27.94" y2="23.368" width="0.4064" layer="1"/>
+<via x="28.575" y="23.368" extent="1-16" drill="0.3"/>
+<via x="28.575" y="24.892" extent="1-16" drill="0.3"/>
+<wire x1="28.575" y1="24.892" x2="28.575" y2="23.368" width="0.4064" layer="1"/>
 <wire x1="36.83" y1="13.97" x2="35.687" y2="13.97" width="0.1524" layer="16"/>
 <via x="35.687" y="13.97" extent="1-16" drill="0.3"/>

Commit message: Push silk changes.
Parts:
- removed LOGO4: OSHW-LOGOS, SparkFun-Aesthetics:OSHW-LOGO-S
- U3, U6: value XC6222B331MR-G -> 3.3V
Other:
- board text added: "4-Layers 1.6mm Thickness 1oz Copper Lead-Free HASL Finish Red Solder Resist White Silkscreen Material: TG155 Stackup: JLC7628"
- board text added: "Alex Brudner"
- board text added: "Revised by:"
- board text added: "v12"
- board text removed: "4-Layers 1.6mm Thickness 1oz Copper Lead-Free HASL Finish Red Solder Resist White Silkscreen"
- board text removed: "v11"
Changed lines of the file:
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@@
 Red Solder Resist
 White Silkscreen
+Material: TG155
+Stackup: JLC7628
 </text>
-<text x="45.72" y="0.381" size="1.778" layer="16" font="vector" ratio="15" rot="SMR0" align="bottom-center">v11</text>
+<text x="45.72" y="0.381" size="1.778" layer="16" font="vector" ratio="15" rot="SMR0" align="bottom-center">v12</text>
 <text x="-1.27" y="43.18" size="1.778" layer="47" font="vector" ratio="15" align="bottom-right">Dimensions
 In Inches</text>
@@
 <text x="1.27" y="0.381" size="1.778" layer="2" font="vector" ratio="15" rot="SR0" align="bottom-center">2</text>
 <text x="1.27" y="0.381" size="1.778" layer="15" font="vector" ratio="15" rot="SMR0" align="bottom-center">3</text>
+<text x="115.57" y="-8.89" size="1.778" layer="51" font="vector" ratio="15">Alex Brudner</text>
+<text x="100.33" y="-8.89" size="1.778" layer="51">Revised by: </text>
 </plain>
 <attributes>
@@
 <attribute name="VALUE" x="21.59" y="10.16" size="0.6096" layer="27"/>
 </element>
-<element name="U3" library="SparkFun-IC-Power" package="SOT23-5" value="XC6222B331MR-G" x="41.275" y="21.59" smashed="yes" rot="R90">
-<attribute name="IOUT" value="700mA" x="41.275" y="21.59" size="1.778" layer="27" rot="R90" display="off"/>
+<element name="U3" library="SparkFun-IC-Power" package="SOT23-5" value="3.3V" x="41.275" y="21.59" smashed="yes" rot="R90">
 <attribute name="NAME" x="39.116" y="19.812" size="0.6096" layer="25" ratio="20" rot="R90"/>
-<attribute name="PROD_ID" value="VREG-16775" x="135.255" y="83.82" size="1.778" layer="27" rot="R90" display="off"/>
-<attribute name="VOUT" value="3.3V" x="41.275" y="21.59" size="1.778" layer="27" rot="R90" display="off"/>
+<attribute name="PROD_ID" value="VREG-12457" x="135.255" y="83.82" size="1.778" layer="27" rot="R90" display="off"/>
+<attribute name="VALUE" value="3.3V" x="41.275" y="21.59" size="1.778" layer="27" rot="R90" display="off"/>
 </element>
 <element name="U4" library="SparkFun-IC-Power" package="DFN-8" value="MAX17048" x="4.953" y="15.875" smashed="yes">
@@
 <attribute name="VALUE" x="6.223" y="13.081" size="0.6096" layer="27" ratio="20"/>
 </element>
-<element name="U6" library="SparkFun-IC-Power" package="SOT23-5" value="XC6222B331MR-G" x="12.7" y="21.59" smashed="yes" rot="R270">
-<attribute name="IOUT" value="700mA" x="12.7" y="21.59" size="1.778" layer="27" rot="R270" display="off"/>
+<element name="U6" library="SparkFun-IC-Power" package="SOT23-5" value="3.3V" x="12.7" y="21.59" smashed="yes" rot="R270">
 <attribute name="NAME" x="14.859" y="23.368" size="0.6096" layer="25" ratio="20" rot="R270"/>
-<attribute name="PROD_ID" value="VREG-16775" x="-81.28" y="-44.45" size="1.778" layer="27" rot="R270" display="off"/>
-<attribute name="VOUT" value="3.3V" x="12.7" y="21.59" size="1.778" layer="27" rot="R270" display="off"/>
+<attribute name="PROD_ID" value="VREG-12457" x="-81.28" y="-44.45" size="1.778" layer="27" rot="R270" display="off"/>
+<attribute name="VALUE" value="3.3V" x="12.7" y="21.59" size="1.778" layer="27" rot="R270" display="off"/>
 </element>
 <element name="U7" library="SparkFun-Sensors" package="LGA-14L" value="ISM330DHCX" x="44.45" y="29.21" smashed="yes">
@@
 <element name="U$42" library="output" package="#35#0" value="" x="18.288" y="27.94" smashed="yes" rot="MR0"/>
 <element name="U$43" library="output" package="#35#0" value="" x="18.288" y="25.4" smashed="yes" rot="MR0"/>
-<element name="LOGO4" library="SparkFun-Aesthetics" package="OSHW-LOGO-S" value="OSHW-LOGOS" x="25.4" y="17.78" smashed="yes" rot="MR0"/>
 <element name="U$45" library="output" package="#SHLD#0" value="" x="34.798" y="5.842" smashed="yes" rot="MR0"/>
 <element name="U$46" library="output" package="#I�C#0" value="" x="36.83" y="11.4935" smashed="yes" rot="MR0"/>
