File: Hardware/SparkFun_DataLogger_IoT_9DOF.sch (EAGLE design)
At the start: 109 parts, among them J10 QWIIC_RIGHT_ANGLE, J3 MICRO-SD-PUSH-PUSH-EXT-PIN, J4 Vertical Qwiic Connector, U1 ESP-WROOM-32E, U10 74HC4066_QUAD_BILATERAL_SWITC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, U2 CH340C, U3 XC6222B331MR-G, U4 MAX17048, U5 MCP73831, U6 XC6222B331MR-G, U7 ISM330DHCX, U8 MMC5983MA_QFN16, U9 74HC4066_QUAD_BILATERAL_SWITC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

Commit message: v11 - SparkFun_DataLogger_IoT_9DOF
Other:
- note added: "v11"
- note removed: "v10"
Changed lines of the file:
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@@
 <text x="106.68" y="233.68" size="2.54" layer="94" font="vector">USB-C</text>
 <text x="350.52" y="10.16" size="2.54" layer="94" font="vector">Paul Clark</text>
-<text x="421.64" y="7.62" size="2.54" layer="94" font="vector">v10</text>
+<text x="421.64" y="7.62" size="2.54" layer="94" font="vector">v11</text>
 <text x="226.06" y="271.78" size="2.54" layer="94" font="vector">Reset and Boot</text>
 <text x="337.82" y="271.78" size="2.54" layer="94" font="vector">LEDs</text>

Commit message: Push silk changes.
Parts:
- removed LOGO4: OSHW-LOGOS, SparkFun-Aesthetics:OSHW-LOGOS
- U3, U6: value XC6222B331MR-G -> 3.3V; device SparkFun-IC-Power:XC6222B331MR-G -> SparkFun-IC-Power:V_REG_AP2112K-3.3V
Other:
- note added: "Revision by: Alex Brudner"
- note added: "Vin Max: 6.0V Iout Max: 600mA Vdo: 250mV @ 600mA Output Discharge: 60Ω Typ"
- note added: "v12"
- note removed: "Vin Max: 6.0V Iout Max: 700mA Vdo: 120mV @ 330mA Output Discharge: 530Ω Typ"
- note removed: "v11"
Changed lines of the file:
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@@
 <setting verticaltext="up"/>
 </settings>
-<grid distance="0.1" unitdist="inch" unit="inch" style="lines" multiple="1" display="no" altdistance="0.05" altunitdist="inch" altunit="inch"/>
+<grid distance="0.1" unitdist="inch" unit="inch" style="lines" multiple="1" display="no" altdistance="0.01" altunitdist="inch" altunit="inch"/>
 <layers>
 <layer number="1" name="Top" color="4" fill="1" visible="no" active="no"/>
@@
 <part name="C5" library="SparkFun-Capacitors" deviceset="2.2UF" device="-0402_TIGHT-10V-10%-X5R" value="2.2uF"/>
 <part name="GND16" library="SparkFun-PowerSymbols" deviceset="GND" device=""/>
-<part name="U3" library="SparkFun-IC-Power" deviceset="XC6222" device="B331MR-G" value="XC6222B331MR-G"/>
+<part name="U3" library="SparkFun-IC-Power" deviceset="V_REG_AP2112" device="K-3.3V" value="3.3V"/>
 <part name="GND17" library="SparkFun-PowerSymbols" deviceset="GND" device=""/>
 <part name="SUPPLY11" library="SparkFun-PowerSymbols" deviceset="3.3V_SW" device=""/>
@@
 <part name="SUPPLY20" library="SparkFun-PowerSymbols" deviceset="V_BATT" device=""/>
 <part name="GND30" library="SparkFun-PowerSymbols" deviceset="GND" device=""/>
-<part name="U6" library="SparkFun-IC-Power" deviceset="XC6222" device="B331MR-G" value="XC6222B331MR-G"/>
+<part name="U6" library="SparkFun-IC-Power" deviceset="V_REG_AP2112" device="K-3.3V" value="3.3V"/>
 <part name="C14" library="SparkFun-Capacitors" deviceset="2.2UF" device="-0402_TIGHT-10V-10%-X5R" value="2.2uF"/>
 <part name="C15" library="SparkFun-Capacitors" deviceset="0.1UF" device="-0402T-6.3V-10%-X7R" value="0.1uF"/>
@@
 <part name="H4" library="SparkFun-Hardware" deviceset="STAND-OFF" device="TIGHT"/>
 <part name="LOGO3" library="SparkFun-Aesthetics" deviceset="QWIIC_LOGO" device="_6MM" value="QWIIC_LOGO_6MM"/>
-<part name="LOGO4" library="SparkFun-Aesthetics" deviceset="OSHW-LOGO" device="S" value="OSHW-LOGOS"/>
 <part name="SUPPLY7" library="SparkFun-PowerSymbols" deviceset="V_USB" device=""/>
 <part name="GND10" library="SparkFun-PowerSymbols" deviceset="GND" device=""/>
@@
 <text x="106.68" y="233.68" size="2.54" layer="94" font="vector">USB-C</text>
 <text x="350.52" y="10.16" size="2.54" layer="94" font="vector">Paul Clark</text>
-<text x="421.64" y="7.62" size="2.54" layer="94" font="vector">v11</text>
+<text x="421.64" y="7.62" size="2.54" layer="94" font="vector">v12</text>
 <text x="226.06" y="271.78" size="2.54" layer="94" font="vector">Reset and Boot</text>
 <text x="337.82" y="271.78" size="2.54" layer="94" font="vector">LEDs</text>
@@
 <text x="48.006" y="272.034" size="1.778" layer="97" font="vector" align="top-center">VDD Range: 3.0V - 3.6V</text>
 <text x="167.386" y="150.114" size="1.778" layer="97" font="vector">Vin Max: 6.0V
-Iout Max: 700mA
-Vdo: 120mV @ 330mA
-Output Discharge: 530Ω Typ</text>
+Iout Max: 600mA
+Vdo: 250mV @ 600mA
+Output Discharge: 60Ω Typ</text>
 <text x="274.32" y="185.42" size="1.778" layer="97" font="vector" align="top-center">If DTR is LOW, toggling RTS from HIGH to LOW resets to run mode.
 If RTS is HIGH, toggling DTR from LOW to HIGH resets to bootloader.</text>
@@
 <wire x1="248.92" y1="127" x2="250.19" y2="125.73" width="0.1524" layer="97"/>
 <text x="383.286" y="213.614" size="1.778" layer="97" font="vector">Vin Max: 6.0V
-Iout Max: 700mA
-Vdo: 120mV @ 330mA
-Output Discharge: 530Ω Typ</text>
+Iout Max: 600mA
+Vdo: 250mV @ 600mA
+Output Discharge: 60Ω Typ</text>
+<text x="332.74" y="6.35" size="2.54" layer="94" font="vector">Revision by: Alex Brudner</text>
 </plain>
 <instances>
@@
 </instance>
 <instance part="H4" gate="G$1" x="426.72" y="30.48" smashed="yes"/>
-<instance part="LOGO3" gate="G$1" x="251.46" y="12.7" smashed="yes"/>
-<instance part="LOGO4" gate="G$1" x="251.46" y="27.94" smashed="yes"/>
+<instance part="LOGO3" gate="G$1" x="251.46" y="17.78" smashed="yes"/>
 <instance part="SUPPLY7" gate="G$1" x="144.78" y="231.14" smashed="yes">
 <attribute name="VALUE" x="144.78" y="233.934" size="1.778" layer="96" align="bottom-center"/>
