File: Hardware/Production/SparkFun_DataLogger_IoT_9DOF-Panel.brd (EAGLE design)
At the start: 115.8 x 161.3 mm, 942 parts, among them J10 QWIIC_RIGHT_ANGLE, J12 MICRO-SD-PUSH-PUSH-EXT-PIN, J13 Vertical Qwiic Connector, J17 QWIIC_RIGHT_ANGLE, J21 MICRO-SD-PUSH-PUSH-EXT-PIN, J22 Vertical Qwiic Connector, J26 QWIIC_RIGHT_ANGLE, J3 MICRO-SD-PUSH-PUSH-EXT-PIN, J30 MICRO-SD-PUSH-PUSH-EXT-PIN, J31 Vertical Qwiic Connector, J35 QWIIC_RIGHT_ANGLE, J39 MICRO-SD-PUSH-PUSH-EXT-PIN, J4 Vertical Qwiic Connector, J40 Vertical Qwiic Connector, J44 QWIIC_RIGHT_ANGLE, J48 MICRO-SD-PUSH-PUSH-EXT-PIN, J49 Vertical Qwiic Connector, J53 QWIIC_RIGHT_ANGLE, U1 ESP-WROOM-32E, U10 74HC4066_QUAD_BILATERAL_SWITC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, U11 74HC4066_QUAD_BILATERAL_SWITC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, U12 ESP-WROOM-32E, U13 CH340C, U14 XC6222B331MR-G, U15 MAX17048, U16 MCP73831, U17 XC6222B331MR-G, U18 ISM330DHCX, U19 MMC5983MA_QFN16, U2 CH340C, U20 74HC4066_QUAD_BILATERAL_SWITC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, U21 74HC4066_QUAD_BILATERAL_SWITC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, U22 ESP-WROOM-32E, U23 CH340C, U24 XC6222B331MR-G, U25 MAX17048, U26 MCP73831, U27 XC6222B331MR-G, U28 ISM330DHCX, U29 MMC5983MA_QFN16, U3 XC6222B331MR-G, U30 74HC4066_QUAD_BILATERAL_SWITC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, U31 74HC4066_QUAD_BILATERAL_SWITC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, U32 ESP-WROOM-32E, U33 CH340C, U34 XC6222B331MR-G, U35 MAX17048, U36 MCP73831, U37 XC6222B331MR-G, U38 ISM330DHCX, U39 MMC5983MA_QFN16, U4 MAX17048, U40 74HC4066_QUAD_BILATERAL_SWITC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, U41 74HC4066_QUAD_BILATERAL_SWITC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, U42 ESP-WROOM-32E, U43 CH340C, U44 XC6222B331MR-G, U45 MAX17048, U46 MCP73831, U47 XC6222B331MR-G, U48 ISM330DHCX, U49 MMC5983MA_QFN16, U5 MCP73831, U50 74HC4066_QUAD_BILATERAL_SWITC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, U51 74HC4066_QUAD_BILATERAL_SWITC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, U52 ESP-WROOM-32E, U53 CH340C, U54 XC6222B331MR-G, U55 MAX17048, U56 MCP73831, U57 XC6222B331MR-G, U58 ISM330DHCX, U59 MMC5983MA_QFN16, U6 XC6222B331MR-G, U60 74HC4066_QUAD_BILATERAL_SWITC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, U7 ISM330DHCX, U8 MMC5983MA_QFN16, U9 74HC4066_QUAD_BILATERAL_SWITC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

Commit message: v11 - SparkFun_DataLogger_IoT_9DOF
Parts:
- added U$295: (no value), output:0_#_BOOT0
- added U$296: (no value), output:RGB0
- added U$297: (no value), output:DATALOGGER0
- added U$298: (no value), output:DATALOGGER1
- added U$299: (no value), output:IOT_9DOF0
- added U$300: (no value), output:IOT_9DOF10
- U$1: device output:OPENLOG0 -> output:IOT_9DOF0
- U$100, U$250: device output:STAT0 -> output:IOT_9DOF10
- U$101, U$151: device output:CHG0 -> output:RESET0
- U$102, U$52: device output:CHG0 -> output:STAT0
- U$103, U$54: device output:STAT0 -> output:CHG0
- U$104, U$153: device output:IMU0 -> output:CHG0
- U$105, U$252: device output:MAG0 -> output:STAT0
- U$106, U$256: device output:X0 -> output:IMU0
- U$107, U$257: device output:Y0 -> output:MAG0
- U$108, U$111, U$258: device output:Z0 -> output:X0
- U$109: device output:X0 -> output:Y0
- U$110: device output:Y0 -> output:Z0
- U$112, U$259: device output:##RESET##0 -> output:Y0
- U$113, U$260: device output:#0_#_#BOOT##0 -> output:Z0
- U$114: device output:#36_#_A0#0 -> output:##RESET##0
- U$115: device output:#39_#_A3#0 -> output:#0_#_#BOOT##0
- U$116: device output:#35_#_A7#0 -> output:#36_#_A0#0
- U$117: device output:#17_#_TXD#0 -> output:#39_#_A3#0
- U$118: device output:#16_#_RXD#0 -> output:#35_#_A7#0
- U$119: device output:#25#0 -> output:#17_#_TXD#0
- U$120: device output:#26#0 -> output:#16_#_RXD#0
- U$121: device output:#SCL#0 -> output:#25#0
- U$122: device output:#SDA#0 -> output:#26#0
- U$123: device output:#3V3_SW#0 -> output:#SCL#0
- U$124: device output:#GND#0 -> output:#SDA#0
- U$125, U$175, U$225: device output:#GND#1 -> output:#3V3_SW#0
- U$126, U$176, U$76: device output:#GND#1 -> output:#GND#0
- U$128, U$177, U$79: device output:#BATT#0 -> output:#GND#1
- U$129, U$178, U$227: device output:#5V#0 -> output:#GND#1
- U$130: device output:#3V3#0 -> output:#BATT#0
- U$131: device output:#33#0 -> output:#5V#0
- U$132: device output:#POCI_#_19#0 -> output:#3V3#0
- U$133: device output:#PICO_#_23#0 -> output:#33#0
- U$134: device output:#SCK_#_18#0 -> output:#POCI_#_19#0
- U$135: device output:#IMU_INT2#0 -> output:#PICO_#_23#0
- U$136: device output:#MAG_INT#0 -> output:#SCK_#_18#0
- U$137, U$187: device output:#35#0 -> output:#IMU_INT2#0
- U$138, U$88: device output:#35#0 -> output:#MAG_INT#0
- U$139, U$90: device output:OPENLOG_ESP320 -> output:#35#0
- U$140, U$189: device output:#SHLD#0 -> output:#35#0
- U$141: device output:#I�C#0 -> output:#SHLD#0
- U$142: device output:STAT_LED0 -> output:#I�C#0
- U$143: device output:RGB_LED0 -> output:STAT_LED0
- U$144: device output:0_#_BOOT0 -> output:RGB_LED0
- U$145: device output:RGB0 -> output:0_#_BOOT0
- U$146: device output:OPENLOG0 -> output:RGB0
- U$147: device output:ESP320 -> output:DATALOGGER0
- U$148: device output:RESET0 -> output:DATALOGGER1
- U$149: device output:STAT0 -> output:IOT_9DOF0
- U$150, U$200: device output:CHG0 -> output:IOT_9DOF10
- U$154, U$203: device output:MAG0 -> output:CHG0
- U$155: device output:X0 -> output:STAT0
- U$156: device output:Y0 -> output:IMU0
- U$157: device output:Z0 -> output:MAG0
- U$161: device output:##RESET##0 -> output:X0
- U$162: device output:#0_#_#BOOT##0 -> output:Y0
- U$163: device output:#36_#_A0#0 -> output:Z0
- U$164: device output:#39_#_A3#0 -> output:##RESET##0
- U$165: device output:#35_#_A7#0 -> output:#0_#_#BOOT##0
- U$166: device output:#17_#_TXD#0 -> output:#36_#_A0#0
- U$167: device output:#16_#_RXD#0 -> output:#39_#_A3#0
- U$168: device output:#25#0 -> output:#35_#_A7#0
- U$169: device output:#26#0 -> output:#17_#_TXD#0
- U$170: device output:#SCL#0 -> output:#16_#_RXD#0
- U$171: device output:#SDA#0 -> output:#25#0
- U$172: device output:#3V3_SW#0 -> output:#26#0
- U$173: device output:#GND#0 -> output:#SCL#0
- U$174, U$224, U$274: device output:#GND#1 -> output:#SDA#0
- U$179, U$228, U$277: device output:#3V3#0 -> output:#GND#1
- U$180: device output:#33#0 -> output:#BATT#0
- U$181: device output:#POCI_#_19#0 -> output:#5V#0
- U$182: device output:#PICO_#_23#0 -> output:#3V3#0
- U$183: device output:#SCK_#_18#0 -> output:#33#0
- U$184: device output:#IMU_INT2#0 -> output:#POCI_#_19#0
- U$185: device output:#MAG_INT#0 -> output:#PICO_#_23#0
- U$186, U$236: device output:#35#0 -> output:#SCK_#_18#0
- U$188: device output:OPENLOG_ESP320 -> output:#MAG_INT#0
- U$190, U$239: device output:#I�C#0 -> output:#35#0
- U$191: device output:STAT_LED0 -> output:#SHLD#0
- U$192: device output:RGB_LED0 -> output:#I�C#0
- U$193: device output:0_#_BOOT0 -> output:STAT_LED0
- U$194: device output:RGB0 -> output:RGB_LED0
- U$195: device output:OPENLOG0 -> output:0_#_BOOT0
- U$196: device output:ESP320 -> output:RGB0
- U$197, U$50: device output:RESET0 -> output:DATALOGGER0
- U$198, U$51: device output:STAT0 -> output:DATALOGGER1
- U$199, U$249: device output:CHG0 -> output:IOT_9DOF0
- U$201: device output:STAT0 -> output:RESET0
- U$202, U$55: device output:IMU0 -> output:STAT0
- U$204, U$253: device output:X0 -> output:CHG0
- U$205: device output:Y0 -> output:STAT0
- U$206: device output:Z0 -> output:IMU0
- U$207, U$57: device output:X0 -> output:MAG0
- U$208, U$58, U$61: device output:Y0 -> output:X0
- U$209, U$59, U$62: device output:Z0 -> output:Y0
- U$210, U$63: device output:##RESET##0 -> output:Z0
- U$211: device output:#0_#_#BOOT##0 -> output:X0
- U$212: device output:#36_#_A0#0 -> output:Y0
- U$213: device output:#39_#_A3#0 -> output:Z0
- U$214: device output:#35_#_A7#0 -> output:##RESET##0
- U$215: device output:#17_#_TXD#0 -> output:#0_#_#BOOT##0
- U$216: device output:#16_#_RXD#0 -> output:#36_#_A0#0
- U$217: device output:#25#0 -> output:#39_#_A3#0
- U$218: device output:#26#0 -> output:#35_#_A7#0
- U$219: device output:#SCL#0 -> output:#17_#_TXD#0
- U$220: device output:#SDA#0 -> output:#16_#_RXD#0
- U$221: device output:#3V3_SW#0 -> output:#25#0
- U$222: device output:#GND#0 -> output:#26#0
- U$223, U$273: device output:#GND#1 -> output:#SCL#0
- U$226: device output:#BATT#0 -> output:#GND#0
- U$229, U$278: device output:#33#0 -> output:#GND#1
- U$230: device output:#POCI_#_19#0 -> output:#BATT#0
- U$231: device output:#PICO_#_23#0 -> output:#5V#0
- U$232: device output:#SCK_#_18#0 -> output:#3V3#0
- U$233: device output:#IMU_INT2#0 -> output:#33#0
- U$234: device output:#MAG_INT#0 -> output:#POCI_#_19#0
- U$235, U$285: device output:#35#0 -> output:#PICO_#_23#0
- U$237: device output:OPENLOG_ESP320 -> output:#IMU_INT2#0
- U$238: device output:#SHLD#0 -> output:#MAG_INT#0
- U$240, U$289: device output:STAT_LED0 -> output:#35#0
- U$241: device output:RGB_LED0 -> output:#SHLD#0
- U$242: device output:0_#_BOOT0 -> output:#I�C#0
- U$243: device output:RGB0 -> output:STAT_LED0
- U$244: device output:OPENLOG0 -> output:RGB_LED0
- U$245: device output:ESP320 -> output:0_#_BOOT0
- U$246: device output:RESET0 -> output:RGB0
- U$247: device output:STAT0 -> output:DATALOGGER0
- U$248: device output:CHG0 -> output:DATALOGGER1
- U$251: device output:IMU0 -> output:RESET0
- U$254: device output:Y0 -> output:CHG0
- U$255: device output:Z0 -> output:STAT0
- U$261: device output:#36_#_A0#0 -> output:X0
- U$262: device output:#39_#_A3#0 -> output:Y0
- U$263: device output:#35_#_A7#0 -> output:Z0
- U$264: device output:#17_#_TXD#0 -> output:##RESET##0
- U$265: device output:#16_#_RXD#0 -> output:#0_#_#BOOT##0
- U$266: device output:#25#0 -> output:#36_#_A0#0
- U$267: device output:#26#0 -> output:#39_#_A3#0
- U$268: device output:#SCL#0 -> output:#35_#_A7#0
- U$269: device output:#SDA#0 -> output:#17_#_TXD#0
- U$270: device output:#3V3_SW#0 -> output:#16_#_RXD#0
- U$271: device output:#GND#0 -> output:#25#0
- U$272: device output:#GND#1 -> output:#26#0
- U$275: device output:#BATT#0 -> output:#3V3_SW#0
- U$276: device output:#5V#0 -> output:#GND#0
- U$279: device output:#POCI_#_19#0 -> output:#GND#1
- U$280: device output:#PICO_#_23#0 -> output:#BATT#0
- U$281: device output:#SCK_#_18#0 -> output:#5V#0
- U$282: device output:#IMU_INT2#0 -> output:#3V3#0
- U$283: device output:#MAG_INT#0 -> output:#33#0
- U$284: device output:#35#0 -> output:#POCI_#_19#0
- U$286: device output:OPENLOG_ESP320 -> output:#SCK_#_18#0
- U$287: device output:#SHLD#0 -> output:#IMU_INT2#0
- U$288: device output:#I�C#0 -> output:#MAG_INT#0
- U$290: device output:RGB_LED0 -> output:#35#0
- U$291: device output:0_#_BOOT0 -> output:#SHLD#0
- U$292: device output:RGB0 -> output:#I�C#0
- U$293: device output:OPENLOG0 -> output:STAT_LED0
- U$294: device output:ESP320 -> output:RGB_LED0
- U$39: device output:ESP320 -> output:RESET0
- U$44: device output:OPENLOG_ESP320 -> output:IOT_9DOF10
- U$56: device output:MAG0 -> output:IMU0
- U$60: device output:X0 -> output:Z0
- U$64: device output:#0_#_#BOOT##0 -> output:##RESET##0
- U$65: device output:#36_#_A0#0 -> output:#0_#_#BOOT##0
- U$66: device output:#39_#_A3#0 -> output:#36_#_A0#0
- U$67: device output:#35_#_A7#0 -> output:#39_#_A3#0
- U$68: device output:#17_#_TXD#0 -> output:#35_#_A7#0
- U$69: device output:#16_#_RXD#0 -> output:#17_#_TXD#0
- U$70: device output:#25#0 -> output:#16_#_RXD#0
- U$71: device output:#26#0 -> output:#25#0
- U$72: device output:#SCL#0 -> output:#26#0
- U$73: device output:#SDA#0 -> output:#SCL#0
- U$74: device output:#3V3_SW#0 -> output:#SDA#0
- U$75: device output:#GND#0 -> output:#3V3_SW#0
- U$80: device output:#5V#0 -> output:#BATT#0
- U$81: device output:#3V3#0 -> output:#5V#0
- U$82: device output:#33#0 -> output:#3V3#0
- U$83: device output:#POCI_#_19#0 -> output:#33#0
- U$84: device output:#PICO_#_23#0 -> output:#POCI_#_19#0
- U$85: device output:#SCK_#_18#0 -> output:#PICO_#_23#0
- U$86: device output:#IMU_INT2#0 -> output:#SCK_#_18#0
- U$87: device output:#MAG_INT#0 -> output:#IMU_INT2#0
- U$97: device output:OPENLOG0 -> output:DATALOGGER0
- U$98: device output:ESP320 -> output:DATALOGGER1
- U$99: device output:RESET0 -> output:IOT_9DOF0
- moved U$199 83.8 mm to (90.6, 69.1), turned to 0 degrees
- moved U$99 78.1 mm to (90.6, 24.1)
- moved U$197 77.6 mm to (90.6, 70.6)
- moved U$200 72.0 mm to (76.7, 65.8), turned to 0 degrees
- moved U$100 70.5 mm to (76.7, 20.8), flipped to the bottom, turned to 0 degrees
- moved U$198 69.6 mm to (76.7, 67.8), flipped to the bottom, turned to 0 degrees
- moved U$176 51.0 mm to (100.1, 51.3)
- moved U$225 50.0 mm to (48.8, 98.8)
- moved U$126 49.2 mm to (48.8, 51.3)
- moved U$274 49.2 mm to (100.1, 101.3)
- moved U$175 48.4 mm to (100.1, 53.8)
- moved U$276 48.4 mm to (100.1, 96.3)
- moved U$224 47.8 mm to (48.8, 101.3)
- moved U$76 47.8 mm to (100.1, 6.35)
- moved U$125 47.4 mm to (48.8, 53.8)
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Other:
- board text added: "v11"
- board text removed: "v10"

Commit message: Push silk changes.
Parts:
- removed LOGO19, LOGO23: SFE_LOGO_NAME.2_INCH, SparkFun-Aesthetics:SFE_LOGO_NAME_.2
- removed LOGO20, LOGO24: SFE_LOGO_FLAME.2_INCH, SparkFun-Aesthetics:SFE_LOGO_FLAME_.2
- removed LOGO21: QWIIC_LOGO_6MM, SparkFun-Aesthetics:QWIIC_6MM
- removed LOGO22: OSHW-LOGOS, SparkFun-Aesthetics:OSHW-LOGO-S
- LOGO10: value OSHW-LOGOS -> QWIIC_LOGO_6MM; device SparkFun-Aesthetics:OSHW-LOGO-S -> SparkFun-Aesthetics:QWIIC_6MM
- LOGO14, LOGO2: value OSHW-LOGOS -> SFE_LOGO_NAME.2_INCH; device SparkFun-Aesthetics:OSHW-LOGO-S -> SparkFun-Aesthetics:SFE_LOGO_NAME_.2
- LOGO15: value SFE_LOGO_NAME.2_INCH -> SFE_LOGO_FLAME.2_INCH; device SparkFun-Aesthetics:SFE_LOGO_NAME_.2 -> SparkFun-Aesthetics:SFE_LOGO_FLAME_.2
- LOGO16: value SFE_LOGO_FLAME.2_INCH -> QWIIC_LOGO_6MM; device SparkFun-Aesthetics:SFE_LOGO_FLAME_.2 -> SparkFun-Aesthetics:QWIIC_6MM
- LOGO17: value QWIIC_LOGO_6MM -> SFE_LOGO_NAME.2_INCH; device SparkFun-Aesthetics:QWIIC_6MM -> SparkFun-Aesthetics:SFE_LOGO_NAME_.2
- LOGO18, LOGO4: value OSHW-LOGOS -> SFE_LOGO_FLAME.2_INCH; device SparkFun-Aesthetics:OSHW-LOGO-S -> SparkFun-Aesthetics:SFE_LOGO_FLAME_.2
- LOGO7: value SFE_LOGO_NAME.2_INCH -> QWIIC_LOGO_6MM; device SparkFun-Aesthetics:SFE_LOGO_NAME_.2 -> SparkFun-Aesthetics:QWIIC_6MM
- LOGO8: value SFE_LOGO_FLAME.2_INCH -> SFE_LOGO_NAME.2_INCH; device SparkFun-Aesthetics:SFE_LOGO_FLAME_.2 -> SparkFun-Aesthetics:SFE_LOGO_NAME_.2
- LOGO9: value QWIIC_LOGO_6MM -> SFE_LOGO_FLAME.2_INCH; device SparkFun-Aesthetics:QWIIC_6MM -> SparkFun-Aesthetics:SFE_LOGO_FLAME_.2
- moved LOGO8 92.6 mm to (25.4, 76.7), flipped to the bottom
- moved LOGO14 78.1 mm to (25.4, 121.7)
- moved LOGO10 72.0 mm to (96.5, 51.8), flipped to the top
- moved LOGO18 71.4 mm to (96.8, 107.7), flipped to the top
- moved LOGO4 71.4 mm to (96.8, 17.8), flipped to the top
- moved LOGO13 68.2 mm to (45.2, 96.8)
- moved LOGO11 51.3 mm to (76.7, 76.7)
- moved LOGO12 51.3 mm to (96.8, 62.7)
- moved LOGO15 44.0 mm to (45.5, 107.7), flipped to the top
- moved LOGO17 40.1 mm to (76.7, 121.7), flipped to the bottom
- moved LOGO7 37.3 mm to (45.2, 51.8), flipped to the top
- moved LOGO16 34.0 mm to (96.5, 96.8)
- moved LOGO2 14.0 mm to (76.7, 31.8)
- moved LOGO9 10.9 mm to (45.5, 62.7)
Other:
- outline, holes or cut-outs redrawn
- board text added: "v12"
- board text removed: "v11"
